Commit message: 修改了turtlebot2和turtlebot2i的启动接口和模型

File: TB2+Kinect2/turtlebot2i_description/urdf/sensors/kinect2.urdf.xacro (robot description, xacro)
@@ -6,5 +6,10 @@
   <!-- Parameterised in part by the values in turtlebot_properties.urdf.xacro -->
   <xacro:macro name="sensor_kinect2" params="parent">
-    <link name="kinect2_model_link">
+    <joint name="camera_mount_joint" type="fixed">
+      <origin xyz="-0.119 0.125 0.306" rpy="${cam_or} ${cam_op} ${cam_oy}"/>
+      <parent link="${parent}"/>
+      <child link="camera_link" />
+    </joint>
+    <link name="camera_link">
       <visual>
        <origin xyz="0 0 0" rpy="-0.11757 0 -1.5707963"/>
@@ -30,15 +35,16 @@
       </inertial>
     </link>
-    <joint name="camera_mount_joint" type="fixed">
-      <origin xyz="-0.13 0.125 0.256" rpy="${cam_or} ${cam_op} ${cam_oy}"/>
-      <parent link="${parent}"/>
-      <child link="kinect2_model_link" />
+    <joint name="camera_rgb_joint" type="fixed">
+      <origin xyz="0.080 -0.2198 0.0317" rpy="${cam_or} ${cam_op} ${cam_oy}"/>
+      <parent link="camera_link"/>
+      <child link="camera_rgb_frame" />
     </joint>
+    <link name="camera_rgb_frame"/>
     <joint name="kinect2_model_joint" type="fixed">
-      <origin xyz="0.080 -0.2198 0.0317" rpy="0 0 0"/>
-      <parent link="kinect2_model_link"/>
-      <child link="kinect2_link" />
+      <origin xyz="0.0 0.0 0.0" rpy="-1.570796327 0.0 -1.570796327"/>
+      <parent link="camera_rgb_frame"/>
+      <child link="camera_rgb_optical_frame" />
     </joint>
-     <link name="kinect2_link"/>
+    <link name="camera_rgb_optical_frame"/>
     <!-- The fixed joints & links below are usually published by static_transformers launched by the OpenNi launch
          files. However, for Gazebo simulation we need them, so we add them here.
@@ -46,12 +52,24 @@
 	<joint name="camera_depth_joint" type="fixed">
 	  <origin xyz="0 0.05 0" rpy="0 0 0" />
-	  <parent link="kinect2_link" />
+	  <parent link="camera_rgb_frame" />
 	  <child link="camera_depth_frame" />
 	</joint>
 	<link name="camera_depth_frame"/>
+	<joint name="camera_ir_joint" type="fixed">
+	  <origin xyz="0 0.05 0" rpy="0 0 0" />
+	  <parent link="camera_rgb_frame" />
+	  <child link="camera_ir_frame" />
+	</joint>
+	<link name="camera_ir_frame"/>
 	<joint name="camera_depth_optical_joint" type="fixed">
-	  <origin xyz="0 0 0" rpy="${-M_PI/2} 0.0 ${-M_PI/2}" />
+	  <origin xyz="0 0 0" rpy="-1.570796327 0.0 -1.570796327" />
 	  <parent link="camera_depth_frame" />
 	  <child link="camera_depth_optical_frame" />
+	</joint>
+	<link name="camera_ir_optical_frame"/>
+	<joint name="camera_ir_optical_joint" type="fixed">
+	  <origin xyz="0 0 0" rpy="-1.570796327 0.0 -1.570796327" />
+	  <parent link="camera_ir_frame" />
+	  <child link="camera_ir_optical_frame" />
 	</joint>
 	<link name="camera_depth_optical_frame"/>

File: TB2+Kinect2/turtlebot_description/robots/kobuki_hexagons_kinect2.urdf.xacro (robot description, xacro)
@@ -8,8 +8,8 @@
   <xacro:include filename="$(find turtlebot_description)/urdf/turtlebot_common_library.urdf.xacro" />
   <xacro:include filename="$(find kobuki_description)/urdf/kobuki.urdf.xacro" />
-  <xacro:include filename="$(find turtlebot_description)/urdf/stacks/hexagons_kinect2.urdf.xacro"/>
+  <xacro:include filename="$(find turtlebot_description)/urdf/stacks/hexagons.urdf.xacro"/>
   <xacro:include filename="$(find turtlebot_description)/urdf/sensors/kinect2.urdf.xacro"/>
   <kobuki/>
-  <stack_hexagons_kinect2 parent="base_link"/>
+  <stack_hexagons parent="base_link"/>
   <sensor_kinect2  parent="base_link"/>
 </robot>
