Commit message: 统一kinect2的坐标系名称，添加kobuki_x_description功能包

File: TB2+Kinect2/kobuki_x_description/urdf/sensors/kinect2_for_kobuki_x.urdf.xacro (robot description, xacro)
@@ -7,5 +7,5 @@
   <xacro:macro name="sensor_kinect2" params="parent">
     <joint name="camera_mount_joint" type="fixed">
-      <origin xyz="-0.119 0.125 0.306" rpy="${cam_or} ${cam_op} ${cam_oy}"/>
+      <origin xyz="-0.15 0.125 0.4526" rpy="${cam_or} ${cam_op} ${cam_oy}"/>
       <parent link="${parent}"/>
       <child link="kinect2_model_link" />

File: TB2+Kinect2/turtlebot_description/urdf/sensors/kinect2.urdf.xacro (robot description, xacro)
@@ -6,4 +6,9 @@
   <!-- Parameterised in part by the values in turtlebot_properties.urdf.xacro -->
   <xacro:macro name="sensor_kinect2" params="parent">
+    <joint name="camera_mount_joint" type="fixed">
+      <origin xyz="-0.13 0.125 0.256" rpy="${cam_or} ${cam_op} ${cam_oy}"/>
+      <parent link="${parent}"/>
+      <child link="kinect2_model_link" />
+    </joint>
     <link name="kinect2_model_link">
       <visual>
@@ -30,32 +35,45 @@
       </inertial>
     </link>
-    <joint name="camera_mount_joint" type="fixed">
-      <origin xyz="-0.13 0.125 0.256" rpy="${cam_or} ${cam_op} ${cam_oy}"/>
-      <parent link="${parent}"/>
-      <child link="kinect2_model_link" />
-    </joint>
-    <joint name="kinect2_model_joint" type="fixed">
+    <joint name="camera_rgb_joint" type="fixed">
       <origin xyz="0.080 -0.2198 0.0317" rpy="0 0 0"/>
       <parent link="kinect2_model_link"/>
-      <child link="kinect2_link" />
+      <child link="camera_rgb_frame" />
     </joint>
-     <link name="kinect2_link"/>
+    <link name="camera_rgb_frame"/>
+    <joint name="camera_rgb_optical_joint" type="fixed">
+      <origin xyz="0.0 0.0 0.0" rpy="-1.570796327 0.0 -1.570796327"/>
+      <parent link="camera_rgb_frame"/>
+      <child link="camera_rgb_optical_frame" />
+    </joint>
+    <link name="camera_rgb_optical_frame"/>
     <!-- The fixed joints & links below are usually published by static_transformers launched by the OpenNi launch
          files. However, for Gazebo simulation we need them, so we add them here.
          (Hence, don't publish them additionally!) -->
-	<joint name="camera_depth_joint" type="fixed">
-	  <origin xyz="0 0.05 0" rpy="0 0 0" />
-	  <parent link="kinect2_link" />
-	  <child link="camera_depth_frame" />
-	</joint>
-	<link name="camera_depth_frame"/>
-	<joint name="camera_depth_optical_joint" type="fixed">
-	  <origin xyz="0 0 0" rpy="${-M_PI/2} 0.0 ${-M_PI/2}" />
-	  <parent link="camera_depth_frame" />
-	  <child link="camera_depth_optical_frame" />
-	</joint>
-	<link name="camera_depth_optical_frame"/>
-	<!-- Kinect sensor for simulation -->
-	<turtlebot_sim_3dsensor/>
+	  <joint name="camera_depth_joint" type="fixed">
+	    <origin xyz="0 0.05 0" rpy="0 0 0" />
+	    <parent link="camera_rgb_frame" />
+	    <child link="camera_depth_frame" />
+	  </joint>
+	  <link name="camera_depth_frame"/>
+	  <joint name="camera_depth_optical_joint" type="fixed">
+	    <origin xyz="0 0 0" rpy="${-M_PI/2} 0.0 ${-M_PI/2}" />
+	    <parent link="camera_depth_frame" />
+	    <child link="camera_depth_optical_frame" />
+	  </joint>
+	  <link name="camera_depth_optical_frame"/>
+	  <joint name="camera_ir_joint" type="fixed">
+	    <origin xyz="0 0.05 0" rpy="0 0 0" />
+	    <parent link="camera_rgb_frame" />
+	    <child link="camera_ir_frame" />
+	  </joint>
+    <link name="camera_ir_frame"/>
+    <joint name="camera_ir_optical_joint" type="fixed">
+	    <origin xyz="0 0 0" rpy="-1.570796327 0.0 -1.570796327" />
+	    <parent link="camera_ir_frame" />
+	    <child link="camera_ir_optical_frame" />
+	  </joint>
+    <link name="camera_ir_optical_frame"/>
+	  <!-- Kinect sensor for simulation -->
+	  <turtlebot_sim_3dsensor/>
   </xacro:macro>
 </robot>
