Commit message: 添加kobuki_xs和astra

File: TB2+Kinect2/kobuki_x_description/urdf/kobuki_xs.urdf.xacro (robot description, xacro)
@@ -1,5 +1,5 @@
 <?xml version="1.0" ?>
-<robot name="kobuki_x" xmlns:xacro="http://ros.org/wiki/xacro">
-    <xacro:macro name="kobuki_x">
+<robot name="kobuki_xs" xmlns:xacro="http://ros.org/wiki/xacro">
+    <xacro:macro name="kobuki_xs">
         <link name="base_footprint"/>
         <joint name="base_joint" type="fixed">
@@ -12,5 +12,5 @@
                 <origin xyz="0.0 0.0 0.0" rpy="1.57079633 0 -1.57079633"/>
                 <geometry>
-                    <mesh filename="package://kobuki_x_description/meshes/kobuki_x.stl" scale="0.001 0.001 0.001"/>
+                    <mesh filename="package://kobuki_x_description/meshes/kobuki_xs.stl" scale="0.001 0.001 0.001"/>
                 </geometry>
                 <material name="light_black">
