Commit message: 修复bug

File: TB2+Kinect2/kobuki_x_description/urdf/bases/kobuki_x.urdf.xacro (robot description, xacro)
@@ -12,5 +12,5 @@
                 <origin xyz="0.0 0.0 0.0" rpy="1.57079633 0 -1.57079633"/>
                 <geometry>
-                    <mesh filename="package://kobuki_x_description/meshes/kobuki_x.stl" scale="0.001 0.001 0.001"/>
+                    <mesh filename="package://kobuki_x_description/meshes/bases/kobuki_x.stl" scale="0.001 0.001 0.001"/>
                 </geometry>
                 <material name="light_black">

File: TB2+Kinect2/kobuki_x_description/urdf/bases/kobuki_xs.urdf.xacro (robot description, xacro)
@@ -13,5 +13,5 @@
                 <origin xyz="0.0 0.0 0.0" rpy="1.57079633 0 -1.57079633"/>
                 <geometry>
-                    <mesh filename="package://kobuki_x_description/meshes/kobuki_xs.stl" scale="0.001 0.001 0.001"/>
+                    <mesh filename="package://kobuki_x_description/meshes/bases/kobuki_xs.stl" scale="0.001 0.001 0.001"/>
                 </geometry>
                 <material name="light_black">

File: TB2+Kinect2/turtlebot_description/robots/kobuki_circle_board_astra.urdf.xacro (robot description, xacro)
@@ -7,5 +7,5 @@
 <robot name="kobuki_x_robot" xmlns:xacro="http://ros.org/wiki/xacro">
   <xacro:include filename="$(find turtlebot_description)/urdf/turtlebot_common_library.urdf.xacro" />
-  <xacro:include filename="$(find kobuki_x_description)/urdf/base/kobuki_xs.urdf.xacro" />
+  <xacro:include filename="$(find kobuki_x_description)/urdf/bases/kobuki_xs.urdf.xacro" />
   <xacro:include filename="$(find kobuki_x_description)/urdf/stacks/circle_board.urdf.xacro"/>
   <xacro:include filename="$(find kobuki_x_description)/urdf/sensors/astra_for_kobuki_xs.urdf.xacro"/>

File: TB2+Kinect2/turtlebot_description/robots/kobuki_circle_board_kinect2.urdf.xacro (robot description, xacro)
@@ -7,5 +7,5 @@
 <robot name="kobuki_x_robot" xmlns:xacro="http://ros.org/wiki/xacro">
   <xacro:include filename="$(find turtlebot_description)/urdf/turtlebot_common_library.urdf.xacro" />
-  <xacro:include filename="$(find kobuki_x_description)/urdf/base/kobuki_xs.urdf.xacro" />
+  <xacro:include filename="$(find kobuki_x_description)/urdf/bases/kobuki_xs.urdf.xacro" />
   <xacro:include filename="$(find kobuki_x_description)/urdf/stacks/circle_board.urdf.xacro"/>
   <xacro:include filename="$(find kobuki_x_description)/urdf/sensors/kinect2_for_kobuki_xs.urdf.xacro"/>

File: TB2+Kinect2/turtlebot_description/robots/kobuki_circle_board_kinect2_rplidar_a2.urdf.xacro (robot description, xacro)
@@ -7,5 +7,5 @@
 <robot name="kobuki_x_robot" xmlns:xacro="http://ros.org/wiki/xacro">
   <xacro:include filename="$(find turtlebot_description)/urdf/turtlebot_common_library.urdf.xacro" />
-  <xacro:include filename="$(find kobuki_x_description)/urdf/base/kobuki_xs.urdf.xacro" />
+  <xacro:include filename="$(find kobuki_x_description)/urdf/bases/kobuki_xs.urdf.xacro" />
   <xacro:include filename="$(find kobuki_x_description)/urdf/stacks/circle_board.urdf.xacro"/>
   <xacro:include filename="$(find kobuki_x_description)/urdf/sensors/kinect2_for_kobuki_xs.urdf.xacro"/>

File: TB2+Kinect2/turtlebot_description/robots/kobuki_twocylinder_kinect2.urdf.xacro (robot description, xacro)
@@ -7,5 +7,5 @@
 <robot name="kobuki_x_robot" xmlns:xacro="http://ros.org/wiki/xacro">
   <xacro:include filename="$(find turtlebot_description)/urdf/turtlebot_common_library.urdf.xacro" />
-  <xacro:include filename="$(find kobuki_x_description)/urdf/base/kobuki_x.urdf.xacro" />
+  <xacro:include filename="$(find kobuki_x_description)/urdf/bases/kobuki_x.urdf.xacro" />
   <xacro:include filename="$(find kobuki_x_description)/urdf/stacks/twocylinder.urdf.xacro"/>
   <xacro:include filename="$(find kobuki_x_description)/urdf/sensors/kinect2_for_kobuki_x.urdf.xacro"/>

Commit message: 添加轮子关节

File: TB2+Kinect2/kobuki_x_description/urdf/bases/kobuki_x.urdf.xacro (robot description, xacro)
@@ -51,4 +51,18 @@
             </visual>
         </link>
+        <joint name="wheel_left_joint" type="continuous">
+            <parent link="base_link"/>
+            <child link="wheel_left_link"/>
+            <origin xyz="0.00 ${0.23/2} 0.0250" rpy="${-M_PI/2} 0 0"/>
+            <axis xyz="0 0 1"/>
+        </joint>
+        <link name="wheel_left_link"/>
+        <joint name="wheel_right_joint" type="continuous">
+            <parent link="base_link"/>
+            <child link="wheel_right_link"/>
+            <origin xyz="0.00 -${0.23/2} 0.0250" rpy="${-M_PI/2} 0 0"/>
+            <axis xyz="0 0 1"/>
+        </joint>
+        <link name="wheel_right_link">
     </xacro:macro>
 </robot>

File: TB2+Kinect2/kobuki_x_description/urdf/bases/kobuki_xs.urdf.xacro (robot description, xacro)
@@ -52,4 +52,18 @@
             </visual>
         </link>
+        <joint name="wheel_left_joint" type="continuous">
+            <parent link="base_link"/>
+            <child link="wheel_left_link"/>
+            <origin xyz="0.00 ${0.23/2} 0.0250" rpy="${-M_PI/2} 0 0"/>
+            <axis xyz="0 0 1"/>
+        </joint>
+        <link name="wheel_left_link"/>
+        <joint name="wheel_right_joint" type="continuous">
+            <parent link="base_link"/>
+            <child link="wheel_right_link"/>
+            <origin xyz="0.00 -${0.23/2} 0.0250" rpy="${-M_PI/2} 0 0"/>
+            <axis xyz="0 0 1"/>
+        </joint>
+        <link name="wheel_right_link">
     </xacro:macro>
 </robot>

Commit message: 修复bug

File: TB2+Kinect2/kobuki_x_description/urdf/bases/kobuki_x.urdf.xacro (robot description, xacro)
@@ -64,5 +64,5 @@
             <axis xyz="0 0 1"/>
         </joint>
-        <link name="wheel_right_link">
+        <link name="wheel_right_link"/>
     </xacro:macro>
 </robot>

File: TB2+Kinect2/kobuki_x_description/urdf/bases/kobuki_xs.urdf.xacro (robot description, xacro)
@@ -65,5 +65,5 @@
             <axis xyz="0 0 1"/>
         </joint>
-        <link name="wheel_right_link">
+        <link name="wheel_right_link"/>
     </xacro:macro>
 </robot>
